File: All_In_One.kicad_pcb (KiCad board)
At the start: 2 copper layers, 106 parts, among them J1 MS_jumper_xaxis, J10 Motors, J11 Fan, J2 MS_jumper_yaxis, J3 Base_Proxy, J4 Water_Pump, J5 MS_jumper, J6 Stepper_xaxis, J7 Stepper_yaxis, J8 Arm_Proxy, J9 bluetooth, Q1 BC547, U1 Prashant_library_Arduino_Mega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, U10 PC817, U11 PC817, U12 PC817, U13 PC817, U14 5V_Regulator, U15 PC817, U16 PC817, U17 PC817, U2 L298, U3 L298, U4 5V_Regulator, U5 PC817, U6 PC817, U7 PC817, U8 PC817, U9 PC817

Commit message: completed joining tracks!
Parts:
- removed A2: Y_AXIS, modFiles:A4998
- removed C1, C15, C29, C31, C35, C4, C6: C, modFiles:Capacitor_Disc_Small
- added R38: R, modFiles:Resistor_small, F.Cu at (193.9, 90.7)
- J3: footprint 0_18:New_conn_1x6 -> 0_18:New_conn_1x4
- J7: value Stepper_yaxis -> servo_motor
- J8: value Arm_Proxy -> ARM PROXY; footprint 0_18:New_conn_1x6 -> 0_18:New_conn_1x4
- R23, R27: value 4k7 -> R
- R4, R6: value 3.3k -> R
- moved J11 140.0 mm to (33.7, 137.6), turned to 180 degrees
- moved J10 94.3 mm to (244.5, 46.9), turned to 0 degrees
- moved U3 76.0 mm to (182.0, 121.5), turned to 180 degrees
- moved R6 75.1 mm to (82.8, 56.3), turned to 90 degrees
- moved R14 74.4 mm to (108.8, 140.2)
- moved U11 74.3 mm to (119.9, 139.8)
- moved R23 74.0 mm to (106.1, 61.4), turned to 270 degrees
- moved C9 73.3 mm to (247.5, 41.1), turned to 0 degrees
- moved R32 72.5 mm to (136.6, 141.2), turned to 90 degrees
- moved J5 71.3 mm to (80.8, 76.3), turned to 90 degrees
- moved J1 70.9 mm to (80.8, 86.3), turned to 90 degrees
- moved J2 70.8 mm to (80.8, 81.4), turned to 90 degrees
- moved J9 70.4 mm to (111.6, 51.0)
- moved R8 65.8 mm to (109.1, 99.0)
- moved U5 65.4 mm to (119.5, 98.5)
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Connections:
- C40 pad 1: Net-(C37-Pad1) -> +12V
- J10 pad 5: /M2_1 -> /M2_2
- J10 pad 6: /M2_2 -> /M2_1
- J10 pad 7: /M3_1 -> /M3_2
- J2 pad 1: /MS3 -> /MS1
- J2 pad 3: /MS1 -> /MS3
- J3 pad 4: Net-(J3-Pad4) -> GND
- J7 pad 1: /Y_2B -> +5V
- J7 pad 2: /Y_2A -> /Servo
- J7 pad 3: /Y_1A -> GND
- J8 pad 3: /P_UP -> +5V
- J8 pad 4: /P_DOWN -> GND
- J9 pad 1: Net-(J9-Pad1) -> Net-(D7-Pad2)
- J9 pad 2: Net-(D7-Pad2) -> Net-(J9-Pad2)
- J9 pad 3: /TX -> GND
- J9 pad 4: GND -> +5V
- R23 pad 1: /P_FRONT1 -> Net-(J9-Pad2)
- R23 pad 2: Net-(J3-Pad3) -> /TX
- R25 pad 2: Net-(J3-Pad4) -> Net-(J3-Pad3)
- R27 pad 1: /P_BACK1 -> +5V
- R27 pad 2: Net-(J3-Pad5) -> +5V
- R4 pad 1: /P_FRONT1 -> +5V
- R4 pad 2: GND -> +5V
- R6 pad 1: /P_BACK1 -> GND
- Rly1 pad 2: +12V -> +5V
- U1 pad 10: /M3_EN -> /M1_EN
- U1 pad 11: /stepy -> Net-(U1-Pad11)
- U1 pad 22: Net-(U1-Pad22) -> /M0_IN2
- U1 pad 23: /M0_IN2 -> /M1_IN1
- U1 pad 25: Net-(U1-Pad25) -> /M1_IN2
- U1 pad 26: Net-(U1-Pad26) -> /M2_IN1
- U1 pad 27: /M2_IN2 -> Net-(U1-Pad27)
- U1 pad 28: /M2_IN1 -> /M2_IN2
- U1 pad 31: /M3_IN1 -> Net-(U1-Pad31)
- U1 pad 32: Net-(U1-Pad32) -> /M3_IN1
- U1 pad 33: /M1_IN2 -> Net-(U1-Pad33)
- U1 pad 34: /M1_IN1 -> Net-(U1-Pad34)
- U1 pad 35: /en_x -> Net-(U1-Pad35)
- U1 pad 36: /en_y -> /en_x
- U1 pad 37: /diry -> Net-(U1-Pad37)
- U1 pad 40: /P_LEFT -> Net-(U1-Pad40)
- U1 pad 41: /P_RIGHT -> /P_LEFT
- U1 pad 42: /P_UP -> Net-(U1-Pad42)
- U1 pad 43: /P_DOWN -> /P_RIGHT
- U1 pad 44: /P_FRONT -> Net-(U1-Pad44)
- U1 pad 45: /P_FRONT1 -> /Servo
- U1 pad 46: /P_BACK -> Net-(U1-Pad46)
- U1 pad 47: /P_BACK1 -> /P_FRONT
- U1 pad 49: Net-(U1-Pad49) -> /P_BACK
- U1 pad 6: /M0_EN -> /M3_EN
- U1 pad 7: /M1_EN -> /M2_EN
- U1 pad 8: /M2_EN -> /M0_EN
- U3 pad 12: /M3_1 -> /M3_2
Routing:
- net Net-(1K12-Pad2): track 0.00 -> 417.1 mm
- net +5V: track 82.3 -> 466.1 mm, vias 0 -> 4
- net /M3_2: track 0.00 -> 213.5 mm, vias 0 -> 2
- net +12V: track 101.6 -> 300.7 mm
- net /M3_1: track 0.00 -> 181.6 mm, vias 0 -> 2
- net +24V: track 0.00 -> 131.0 mm, vias 0 -> 2
- net /1_2: track 0.00 -> 121.6 mm
- net /1_1: track 0.00 -> 121.3 mm
- net /0_1: track 0.00 -> 111.8 mm
- net /0_2: track 0.00 -> 111.0 mm
- net /M0_1: track 0.00 -> 103.8 mm
- net /M0_2: track 0.00 -> 101.6 mm
- net /1_E: track 0.00 -> 76.8 mm
- net /M2_2: track 0.00 -> 73.6 mm
- net /M2_1: track 0.00 -> 71.0 mm
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- added copper zone on B.Cu, net GND
- added copper zone on B.Cu, net gnd

Commit message: completed circuit
Parts:
- J9: footprint modFiles:bluetooth -> 0_18:bluetooth
- R7: value 1.5k -> 470
- U14: footprint modFiles:Buck 5A -> modFiles:Buck_Regulator
- U4: footprint modFiles:Buck_Regulator -> modFiles:Buck_5A
- moved C38 55.0 mm to (199.1, 84.8), turned to 0 degrees
- moved J10 48.9 mm to (208.4, 79.9)
- moved D8 48.6 mm to (199.6, 120.4), turned to 0 degrees
- moved C9 47.6 mm to (199.9, 43.2), turned to 180 degrees
- moved F2 46.2 mm to (196.9, 135.8), turned to 270 degrees
- moved U14 45.0 mm to (204.7, 78.9), turned to 90 degrees
- moved d2 44.5 mm to (212.9, 138.9), turned to 0 degrees
- moved C39 38.5 mm to (199.6, 93.7), turned to 0 degrees
- moved R35 35.1 mm to (205.6, 120.1), turned to 270 degrees
- moved C41 33.1 mm to (199.4, 102.9), turned to 0 degrees
- moved U4 16.3 mm to (39.4, 61.3), turned to 90 degrees
- moved R38 16.0 mm to (178.0, 89.6)
- moved R28 14.3 mm to (131.8, 83.5)
- moved R20 14.1 mm to (46.9, 45.0), turned to 180 degrees
- moved U2 13.6 mm to (169.4, 60.3)
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- renumbered C40 to 1000uf, C42 to 10uf, J1 to 5V, J5 to GND, J2 to MS1
Connections:
- C9 pad 2: Net-(C9-Pad2) -> gnd
- J10 pad 1: /M0_1 -> /M1_2
- J10 pad 2: /M0_2 -> /M1_1
- J10 pad 3: /M1_1 -> /M0_2
- J10 pad 4: /M1_2 -> /M0_1
- J10 pad 7: /M3_2 -> /M3_1
- J10 pad 8: /M3_1 -> /M3_2
- J9 pad 1: Net-(D7-Pad2) -> /state
- J9 pad 2: Net-(J9-Pad2) -> Net-(D7-Pad2)
- J9 pad 3: GND -> Net-(J9-Pad3)
- J9 pad 4: +5V -> GND
- R23 pad 1: Net-(J9-Pad2) -> Net-(J9-Pad3)
- U1 pad 11: Net-(U1-Pad11) -> /state
- U14 pad 1: Net-(1K12-Pad2) -> +24V
- U14 pad 2: Net-(C9-Pad2) -> gnd
- U14 pad 4: +24V -> Net-(1K12-Pad2)
Routing:
- net +5V: track 466.1 -> 544.3 mm
- net +24V: track 131.0 -> 192.0 mm, vias 2 -> 0
- net /M2_2: track 73.6 -> 21.6 mm
- net /M2_1: track 71.0 -> 21.2 mm
- net Net-(1K12-Pad2): track 417.1 -> 381.9 mm
- net /M0_1: track 103.8 -> 138.9 mm
- net /M3_2: track 213.5 -> 179.3 mm
- net /M0_2: track 101.6 -> 130.6 mm
- net /M3_1: track 181.6 -> 156.4 mm
- net Net-(C9-Pad2): track 21.8 -> 0.00 mm
- net /M1_1: track 45.9 -> 64.6 mm
- net Net-(J9-Pad3): track 0.00 -> 18.0 mm
- net /1_E: track 76.8 -> 61.0 mm
- net Net-(J9-Pad2): track 14.8 -> 0.00 mm
- net /0_2: track 111.0 -> 96.4 mm
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Other:
- board text added: "12V"
- board text added: "24V"
- board text added: "5V_2A"
- board text added: "5V_3A"
- board text added: "GND"
- board text added: "GND 12V FAN"
- board text added: "GND DIR 5V STEP"
- board text added: "GND POW P_RIGHT P_LEFT ARM_PROXY"
- board text added: "GND POW WATER_PUMP"
- board text added: "GND PWM POW SERVO"
- board text added: "GND P_BACK P_FRONT POW BASE_PROXY"
- board text added: "M3_2 M3_1 M2_1 M2_2 M0_1 M0_2 M1_1 M1_2"
- board text added: "MS1 MS2 MS3"
- board text added: "X_1B X_1A X_2A X_2B STEPPER"
- board text added: "gnd"

Commit message: completed circuit1
Parts:
- added C1: CP1, modFiles:Capacitor_1000uF, F.Cu at (40.9, 84.1)
- added R39: R, modFiles:Resistor_small, F.Cu at (144.3, 126.7)
- added R40: R, modFiles:Resistor_small, F.Cu at (147.8, 126.0)
- moved C36 42.9 mm to (79.9, 109.1), turned to 90 degrees
- moved 10uf 25.4 mm to (33.8, 53.8)
- moved C37 24.7 mm to (32.8, 61.0)
- moved C3 20.5 mm to (89.4, 93.2)
- moved C2 15.3 mm to (63.2, 133.1)
- moved C13 10.2 mm to (87.2, 97.3)
- moved C33 8.68 mm to (84.6, 72.4), turned to 90 degrees
- moved R35 8.56 mm to (212.7, 125.0), turned to 180 degrees
- moved D8 8.17 mm to (207.8, 119.5)
- moved J10 6.41 mm to (214.8, 79.5)
- moved D2 2.87 mm to (45.2, 105.5), turned to 180 degrees
- moved d1 2.58 mm to (29.5, 72.1)
- moved R23 2.19 mm to (105.2, 59.4)
- moved R38 2.09 mm to (176.3, 88.4)
- moved R2 1.47 mm to (38.1, 122.2)
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Routing:
- net +5V: track 544.3 -> 481.2 mm
- net gnd: track 37.8 -> 88.6 mm, vias 2 -> 0
- net GND: track 60.2 -> 97.6 mm
- net +12V: track 294.1 -> 318.4 mm
- net Net-(1K12-Pad2): track 381.9 -> 360.5 mm
- net Net-(C36-Pad1): track 69.3 -> 89.0 mm
- net +24V: track 192.0 -> 172.6 mm
- net Net-(C37-Pad1): track 50.9 -> 36.1 mm
- net /dirx: track 57.5 -> 70.5 mm
- net /M3_2: track 179.3 -> 167.9 mm, vias 2 -> 0
- net /1_2: track 112.2 -> 104.4 mm
- net /M2_1: track 21.2 -> 27.7 mm
- net /M2_2: track 21.6 -> 28.2 mm
- net /M1_2: track 53.2 -> 47.2 mm
- net /M1_1: track 64.6 -> 58.8 mm
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
Commit message: battery indicator
Parts:
- added C4: C, modFiles:Capacitor_Disc_Small, F.Cu at (-9.69, 52.1)
- added C6: C, modFiles:Capacitor_Disc_Small, F.Cu at (196.6, 49.4)
- added D12: D_Zener, Diode_THT:D_T-1_P5.08mm_Horizontal, F.Cu at (-21.8, 52.8)
- added D13: RED, modFiles:LED_D3.0mm, F.Cu at (163.2, 26.2)
- added D14: D_Zener, Diode_THT:D_T-1_P5.08mm_Horizontal, F.Cu at (196.1, 42.3)
- added D15: RED, modFiles:LED_D3.0mm, F.Cu at (138.0, 26.2)
- added D16: RED, modFiles:LED_D3.0mm, F.Cu at (152.5, 26.2)
- added D4: RED, modFiles:LED_D3.0mm, F.Cu at (30.4, 27.7)
- added D5: RED, modFiles:LED_D3.0mm, F.Cu at (20.0, 27.6)
- added D6: RED, modFiles:LED_D3.0mm, F.Cu at (38.9, 27.9)
- added J12: Raspberry_pi, 0_18:New_conn_1x2, F.Cu at (-21.4, 30.6)
- added Q2: BC547, Package_TO_SOT_THT:TO-92_Inline, F.Cu at (31.3, 32.1)
- added Q3: BC547, Package_TO_SOT_THT:TO-92_Inline, F.Cu at (21.1, 32.7)
- added Q4: BC547, Package_TO_SOT_THT:TO-92_Inline, F.Cu at (39.8, 32.3)
- added Q5: BC547, Package_TO_SOT_THT:TO-92_Inline, F.Cu at (161.4, 31.0)
- added Q6: BC547, Package_TO_SOT_THT:TO-92_Inline, F.Cu at (138.5, 31.5)
- added Q7: BC547, Package_TO_SOT_THT:TO-92_Inline, F.Cu at (152.5, 30.8)
- added R41: 4.7k, modFiles:Resistor_small, F.Cu at (5.50, 64.4)
- added R42: 4.7k, modFiles:Resistor_small, F.Cu at (-16.1, 55.5)
- added R43: 470, modFiles:Resistor_small, F.Cu at (26.5, 39.1)
- added R44: 10K, modFiles:Resistor_small, F.Cu at (-2.94, 32.0)
- added R45: 470, modFiles:Resistor_small, F.Cu at (16.9, 38.8)
- added R46: 39K, modFiles:Resistor_small, F.Cu at (-16.5, 42.4)
- added R47: 470, modFiles:Resistor_small, F.Cu at (44.8, 36.2)
- added R48: 680, modFiles:Resistor_small, F.Cu at (-13.8, 39.4)
- added R49: 1K, modFiles:Resistor_small, F.Cu at (-9.78, 31.9)
- added R50: 470, modFiles:Resistor_small, F.Cu at (-16.4, 28.9)
- added R51: 330, modFiles:Resistor_small, F.Cu at (4.88, 35.7)
- added R52: 39K, modFiles:Resistor_small, F.Cu at (-13.1, 42.4)
- added R53: 10K, modFiles:Resistor_small, F.Cu at (4.79, 28.5)
- added R54: 10K, modFiles:Resistor_small, F.Cu at (5.51, 46.4)
- added R55: 1K, modFiles:Resistor_small, F.Cu at (-21.9, 42.4)
- added R56: 4.7k, modFiles:Resistor_small, F.Cu at (-13.0, 59.1)
- added R57: 470, modFiles:Resistor_small, F.Cu at (58.7, 143.3)
- added R59: 220, modFiles:Resistor_small, F.Cu at (205.7, 35.3)
- added R60: 4.7k, modFiles:Resistor_small, F.Cu at (213.1, 30.5)
- added R61: 47, modFiles:Resistor_small, F.Cu at (205.6, 26.0)
- added R62: 100, modFiles:Resistor_small, F.Cu at (202.6, 26.1)
- added R63: 1k, modFiles:Resistor_small, F.Cu at (195.0, 32.0)
- added R64: 4.7k, modFiles:Resistor_small, F.Cu at (132.2, 26.8)
- added R65: 4.7k, modFiles:Resistor_small, F.Cu at (166.4, 34.2)
- added R67: 10K, modFiles:Resistor_small, F.Cu at (184.7, 36.5)
- added R68: 10K, modFiles:Resistor_small, F.Cu at (181.8, 36.6)
- added R69: 2.2k, modFiles:Resistor_small, F.Cu at (193.1, 47.1)
- added R70: 4.7k, modFiles:Resistor_small, F.Cu at (145.6, 37.1)
- added R71: 470, modFiles:Resistor_small, F.Cu at (170.0, 34.3)
- added R72: 470, modFiles:Resistor_small, F.Cu at (128.8, 34.3)
- added R73: 470, modFiles:Resistor_small, F.Cu at (148.9, 37.1)
- added U18: LM339, Package_DIP:DIP-14_W7.62mm_LongPads, F.Cu at (2.16, 55.4)
- added U19: LM339, Package_DIP:DIP-14_W7.62mm_LongPads, F.Cu at (176.7, 33.1)
- added U20: 5V_Regulator, modFiles:Buck_5A, F.Cu at (-5.61, 72.7)
- moved C9 26.6 mm to (222.8, 29.5)
- moved d1 3.85 mm to (28.0, 75.7)
- moved J11 1.49 mm to (33.3, 136.1)
- moved J6 1.47 mm to (33.1, 111.8)
- moved J4 1.47 mm to (33.4, 124.0)
- moved J3 1.23 mm to (59.2, 134.3)
- moved C1 0.65 mm to (41.5, 84.1)
- moved J7 0.39 mm to (79.8, 135.3)
Connections:
- U4 pad 1: +12V -> GND
- U4 pad 2: GND -> +12V
- U4 pad 3: GND -> +5V
- U4 pad 4: +5V -> GND
Routing:
- net +12V: track 318.4 -> 618.8 mm
- net Net-(1K12-Pad2): track 360.5 -> 517.7 mm
- net +24V: track 172.6 -> 267.3 mm, vias 0 -> 2
- net /X3: track 0.00 -> 79.9 mm
- net /X2: track 0.00 -> 62.0 mm
- net Net-(J12-Pad1): track 0.00 -> 55.7 mm
- net /B_X1: track 0.00 -> 52.5 mm
- net +5V: track 481.2 -> 527.6 mm
- net /B_X2: track 0.00 -> 37.8 mm
- net /X1: track 0.00 -> 37.8 mm
- net /B_V3: track 0.00 -> 37.3 mm
- net /Z: track 0.00 -> 29.2 mm, vias 0 -> 2
- net /B_X3: track 0.00 -> 26.2 mm
- net Net-(R53-Pad1): track 0.00 -> 23.8 mm
- net Net-(R50-Pad1): track 0.00 -> 21.6 mm
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
Commit message: added buck for pi
Parts:
- added R58: 470, modFiles:Resistor_small, F.Cu at (251.5, 63.5)
- moved J12 168.1 mm to (146.5, 38.6), turned to 90 degrees
- moved R50 65.0 mm to (48.6, 28.4), turned to 180 degrees
- moved C4 61.4 mm to (48.2, 31.7), turned to 180 degrees
- moved R51 55.2 mm to (59.5, 28.0)
- moved R44 54.8 mm to (51.9, 31.3)
- moved D12 54.6 mm to (32.5, 46.7)
- moved R53 53.6 mm to (58.0, 34.7)
- moved R49 50.7 mm to (40.3, 39.3), turned to 90 degrees
- moved R48 50.6 mm to (36.8, 39.3)
- moved C5 49.7 mm to (88.9, 128.7)
- moved C7 49.6 mm to (94.1, 121.5)
- moved R56 48.6 mm to (35.2, 65.2), turned to 90 degrees
- moved R42 48.5 mm to (31.4, 65.2), turned to 90 degrees
- moved U20 48.3 mm to (42.5, 76.6)
- moved Q1 48.1 mm to (87.2, 113.6)
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- renumbered R70 to eR70
Connections:
- J12 pad 1: Net-(J12-Pad1) -> GND
- U20 pad 4: Net-(J12-Pad1) -> GND
Routing:
- net Net-(J12-Pad2): track 21.4 -> 160.1 mm
- net GND: track 97.8 -> 180.2 mm
- net Net-(J12-Pad1): track 55.7 -> 0.00 mm
- net gnd: track 88.6 -> 140.7 mm
- net Net-(1K12-Pad2): track 517.7 -> 555.2 mm
- net +5V: track 527.6 -> 553.0 mm
- net Net-(R50-Pad1): track 21.6 -> 3.45 mm
- net /X_2B: track 55.7 -> 70.6 mm
- net Net-(C36-Pad1): track 87.8 -> 101.3 mm
- net /X_2A: track 48.6 -> 61.6 mm
- net /V1: track 9.39 -> 21.4 mm
- net +12V: track 618.8 -> 607.4 mm
- net /X_1A: track 42.3 -> 53.3 mm
- net /V3: track 14.1 -> 23.3 mm
- net Net-(D4-Pad2): track 13.3 -> 4.46 mm
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Other:
- board outline added: 257.1 x 139.3 mm
- board text added: "5V GND PI"

Commit message: completed board!
Parts:
- added R66: R, modFiles:Resistor_small, F.Cu at (157.1, 84.0)
- added R74: R, modFiles:Resistor_small, F.Cu at (146.2, 78.7)
- Q1, Q5, Q6, Q7: footprint Package_TO_SOT_THT:TO-92_Inline -> modFiles:BC547
- Q2, Q3, Q4: footprint Package_TO_SOT_THT:TO-92_Inline -> modFiles:BC547; moved to B.Cu
- R44: value 10K -> 1K
- R46, R52: value 39K -> 3.9K
- R48: value 680 -> 68
- R49: value 1K -> 100
- R50: value 470 -> 47
- R51: value 330 -> 33
- moved D7 18.6 mm to (146.2, 85.9)
- moved C6 16.4 mm to (224.4, 50.2), turned to 0 degrees
- moved D12 14.8 mm to (42.8, 36.1), turned to 0 degrees
- moved eR70 10.5 mm to (200.3, 39.6)
- moved R64 8.52 mm to (184.2, 32.9)
- moved R55 8.47 mm to (33.1, 39.7)
- moved R72 8.33 mm to (180.6, 40.5)
- moved Q6 7.33 mm to (175.4, 33.4)
- moved Q7 5.69 mm to (190.9, 33.8)
- moved D14 4.21 mm to (239.1, 49.2), turned to 90 degrees
- moved D16 4.04 mm to (192.6, 29.3), turned to 0 degrees
- moved R73 3.55 mm to (196.6, 39.8)
- moved R49 3.32 mm to (38.1, 36.9)
- moved R48 3.08 mm to (35.0, 36.8)
- moved R69 3.00 mm to (237.2, 52.9)
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Connections:
- D12 pad 1: Net-(D12-Pad1) -> /Z
- D14 pad 1: Net-(D14-Pad1) -> /B_Z
- J9 pad 2: Net-(D7-Pad2) -> Net-(J9-Pad2)
- R55 pad 2: Net-(D12-Pad1) -> /Z
- R69 pad 2: Net-(D14-Pad1) -> /B_Z
Routing:
- net GND: track 180.2 -> 215.9 mm
- net Net-(1K12-Pad2): track 555.2 -> 528.0 mm
- net /B_Z: track 17.3 -> 41.2 mm
- net gnd: track 140.7 -> 156.9 mm
- net +24V: track 269.4 -> 283.9 mm, vias 2 -> 1
- net Net-(J9-Pad2): track 0.00 -> 12.9 mm
- net Net-(D15-Pad2): track 14.2 -> 4.77 mm
- net /Z: track 29.2 -> 38.4 mm
- net Net-(D7-Pad2): track 12.9 -> 4.55 mm
- net Net-(D14-Pad1): track 8.16 -> 0.00 mm
- net Net-(R59-Pad1): track 9.99 -> 3.96 mm
- net /V2: track 24.6 -> 20.4 mm
- net Net-(D12-Pad1): track 3.77 -> 0.00 mm
- net /B_X1: track 52.5 -> 55.8 mm
- net /RX: track 9.96 -> 7.60 mm
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
Commit message: finalized board
Parts:
- added J13: Conn_01x01_Female, Connector_PinHeader_2.00mm:PinHeader_1x01_P2.00mm_Vertical, F.Cu at (43.7, 46.4)
- added J13: Conn_01x01_Female, Connector_PinHeader_2.00mm:PinHeader_1x01_P2.00mm_Vertical, F.Cu at (43.7, 55.1)
Other:
- board text added: "EXTREMELY LOW"
- board text added: "LOW"
- board text added: "TOO LOW"
Changed lines of the file:
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@@
   (general
     (thickness 1.6)
-    (drawings 36)
+    (drawings 44)
     (tracks 1553)
     (zones 0)
-    (modules 156)
+    (modules 158)
     (nets 163)
   )
@@
   )
   (setup
-    (last_trace_width 1.2)
+    (last_trace_width 0.25)
     (user_trace_width 0.5)
     (user_trace_width 0.8)
@@
     (add_net gnd)
   )
+  (module Connector_PinHeader_2.00mm:PinHeader_1x01_P2.00mm_Vertical (layer F.Cu)
+    (at 43.684 46.434 90)
+    (descr "Through hole straight pin header, 1x01, 2.00mm pitch, single row")
+    (tags "Through hole pin header THT 1x01 2.00mm single row")
+    (fp_text reference J13 (at 0 -2.06 90) (layer F.SilkS)
+      (effects (font (size 1 1) (thickness 0.15)))
+    )
+    (fp_text value Conn_01x01_Female (at 0 2.06 90) (layer F.Fab)
+      (effects (font (size 1 1) (thickness 0.15)))
+    )
+    (pad 1 thru_hole oval (at 0 0 90) (size 2 1.35) (drill 0.8) (layers *.Cu *.Mask)
+      (net 143 /Z))
+    (model ${KISYS3DMOD}/Connector_PinHeader_2.00mm.3dshapes/PinHeader_1x01_P2.00mm_Vertical.wrl
+      (at (xyz 0 0 0))
+      (scale (xyz 1 1 1))
+      (rotate (xyz 0 0 0))
+    )
+  )
+  (module Connector_PinHeader_2.00mm:PinHeader_1x01_P2.00mm_Vertical (layer F.Cu)
+    (at 43.684 55.07 90)
+    (descr "Through hole straight pin header, 1x01, 2.00mm pitch, single row")
+    (tags "Through hole pin header THT 1x01 2.00mm single row")
+    (fp_text reference J13 (at 0 -2.06 90) (layer F.SilkS)
+      (effects (font (size 1 1) (thickness 0.15)))
+    )
+    (fp_text value Conn_01x01_Female (at 0 2.06 90) (layer F.Fab)
+      (effects (font (size 1 1) (thickness 0.15)))
+    )
+    (pad 1 thru_hole oval (at 0 0 90) (size 2 1.35) (drill 0.8) (layers *.Cu *.Mask)
+      (net 143 /Z))
+    (model ${KISYS3DMOD}/Connector_PinHeader_2.00mm.3dshapes/PinHeader_1x01_P2.00mm_Vertical.wrl
+      (at (xyz 0 0 0))
+      (scale (xyz 1 1 1))
+      (rotate (xyz 0 0 0))
+    )
+  )
   (module modFiles:Resistor_small (layer F.Cu)
     (at 146.25 78.74 270)
@@
     )
   )
+  (gr_text LOW (at 182.114 25.352 180) (layer F.SilkS)
+    (effects (font (size 1.5 1.5) (thickness 0.3)))
+  )
+  (gr_text "TOO LOW" (at 193.544 25.352 180) (layer F.SilkS)
+    (effects (font (size 1.5 1) (thickness 0.25)))
+  )
+  (gr_text "EXTREMELY\nLOW" (at 206.498 24.082 180) (layer F.SilkS)
+    (effects (font (size 1.5 1) (thickness 0.25)))
+  )
+  (gr_text 12V (at 74.672 22.304 180) (layer F.SilkS)
+    (effects (font (size 2 2) (thickness 0.3)))
+  )
+  (gr_text "24V\n" (at 195.068 21.288 180) (layer F.SilkS)
+    (effects (font (size 2 2) (thickness 0.3)))
+  )
+  (gr_text "EXTREMELY\nLOW" (at 65.782 25.606 180) (layer F.SilkS)
+    (effects (font (size 1.5 1) (thickness 0.25)))
+  )
+  (gr_text "TOO LOW" (at 74.164 26.622 180) (layer F.SilkS)
+    (effects (font (size 1.5 1) (thickness 0.25)))
+  )
+  (gr_text LOW (at 82.292 25.86 180) (layer F.SilkS)
+    (effects (font (size 1.5 1.5) (thickness 0.3)))
+  )
   (gr_line (start 23 77.43) (end 23.08 19.67) (angle 90) (layer F.SilkS) (width 0.2))
