File: All_In_One.sch (KiCad schematic (older format))
At the start: 154 parts, among them J1 MS_jumper_xaxis, J10 Motors, J11 Fan, J12 Raspberry_pi, J2 MS_jumper_yaxis, J3 Base_Proxy, J4 Water_Pump, J5 MS_jumper, J6 Stepper_xaxis, J7 servo_motor, J8 ARM PROXY, J9 bluetooth, Q1 BC547, Q2 BC547, Q3 BC547, Q4 BC547, Q5 BC547, Q6 BC547, Q7 BC547, U1 Prashant_library_Arduino_Mega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, U10 PC817, U11 PC817, U12 PC817, U13 PC817, U14 5V_Regulator, U15 PC817, U16 PC817, U17 PC817, U18 LM339, U19 LM339, U2 L298, U20 5V_Regulator, U3 L298, U4 5V_Regulator, U5 PC817, U6 PC817, U7 PC817, U8 PC817, U9 PC817

Commit message: completed board!
Parts:
- added R66, R74: R, modFiles:Resistor_small, symbol Device:R
- Q1, Q2, Q3, Q4, Q5, Q6, Q7: footprint Package_TO_SOT_THT:TO-92_Inline -> modFiles:BC547
- R44: value 10K -> 1K
- R46, R52: value 39K -> 3.9K
- R48: value 680 -> 68
- R49: value 1K -> 100
- R50: value 470 -> 47
- R51: value 330 -> 33
Connections:
- net B_Z: now also D14.1 (K), R69.2
- net GND: now also R66.1
- net RX: now also R74.2
- net Z: now also D12.1 (K), R55.2
- net at J9.2 (Pin_2): now also R74.1; no longer D7.2 (A)
- new net: D7.2 (A), R66.2
Changed lines of the file:
@@
 L Device:D_Zener D7
 U 1 1 5F466363
-P 4550 900
-F 0 "D7" H 4550 1116 50  0001 C CNN
-F 1 "D_Zener" H 4550 1025 50  0001 C CNN
-F 2 "Diode_THT:D_T-1_P5.08mm_Horizontal" H 4550 900 50  0001 C CNN
-F 3 "~" H 4550 900 50  0001 C CNN
-	1    4550 900
-	1    0    0    -1
+P 4250 1050
+F 0 "D7" H 4250 1266 50  0001 C CNN
+F 1 "D_Zener" H 4250 1175 50  0001 C CNN
+F 2 "Diode_THT:D_T-1_P5.08mm_Horizontal" H 4250 1050 50  0001 C CNN
+F 3 "~" H 4250 1050 50  0001 C CNN
+	1    4250 1050
+	0    1    1    0
 $EndComp
 $Comp
@@
 $EndComp
 Wire Wire Line
-	4400 900  4250 900
-Wire Wire Line
 	4250 900  4250 800
 Text Label 7350 5300 2    50   ~ 0
@@
 F 0 "Q1" H 5291 7546 50  0001 L CNN
 F 1 "BC547" H 4800 7550 50  0000 L CNN
-F 2 "Package_TO_SOT_THT:TO-92_Inline" H 5300 7425 50  0001 L CIN
+F 2 "modFiles:BC547" H 5300 7425 50  0001 L CIN
 F 3 "http://www.fairchildsemi.com/ds/BC/BC547.pdf" H 5100 7500 50  0001 L CNN
 	1    5100 7500
@@
 	4750 1200 4850 1200
 Wire Wire Line
-	4850 1100 4600 1100
+	4850 1100 4700 1100
 Wire Wire Line
 	4850 1000 4400 1000
-Wire Wire Line
-	4850 900  4700 900
 Text Label 4850 800  2    50   ~ 0
 state
@@
 F 0 "Q3" H 3041 6796 50  0001 L CNN
 F 1 "BC547" H 2550 6950 50  0000 L CNN
-F 2 "Package_TO_SOT_THT:TO-92_Inline" H 3050 6675 50  0001 L CIN
+F 2 "modFiles:BC547" H 3050 6675 50  0001 L CIN
 F 3 "http://www.fairchildsemi.com/ds/BC/BC547.pdf" H 2850 6750 50  0001 L CNN
 	1    2850 6750
@@
 F 0 "Q4" H 3291 7396 50  0001 L CNN
 F 1 "BC547" H 2800 7550 50  0000 L CNN
-F 2 "Package_TO_SOT_THT:TO-92_Inline" H 3300 7275 50  0001 L CIN
+F 2 "modFiles:BC547" H 3300 7275 50  0001 L CIN
 F 3 "http://www.fairchildsemi.com/ds/BC/BC547.pdf" H 3100 7350 50  0001 L CNN
 	1    3100 7350
@@
 F 0 "Q2" H 2041 7546 50  0001 L CNN
 F 1 "BC547" H 1550 7700 50  0000 L CNN
-F 2 "Package_TO_SOT_THT:TO-92_Inline" H 2050 7425 50  0001 L CIN
+F 2 "modFiles:BC547" H 2050 7425 50  0001 L CIN
 F 3 "http://www.fairchildsemi.com/ds/BC/BC547.pdf" H 1850 7500 50  0001 L CNN
 	1    1850 7500
@@
 P 3600 4500
 F 0 "R46" V 3680 4500 50  0000 C CNN
-F 1 "39K" V 3600 4500 50  0000 C CNN
+F 1 "3.9K" V 3600 4500 50  0000 C CNN
 F 2 "modFiles:Resistor_small" V 3530 4500 50  0001 C CNN
 F 3 "~" H 3600 4500 50  0001 C CNN
@@
 P 3850 4500
 F 0 "R52" V 3930 4500 50  0000 C CNN
-F 1 "39K" V 3850 4500 50  0000 C CNN
+F 1 "3.9K" V 3850 4500 50  0000 C CNN
 F 2 "modFiles:Resistor_small" V 3780 4500 50  0001 C CNN
 F 3 "~" H 3850 4500 50  0001 C CNN
@@
 P 3750 4800
 F 0 "R48" V 3830 4800 50  0000 C CNN
-F 1 "680" V 3750 4800 50  0000 C CNN
+F 1 "68" V 3750 4800 50  0000 C CNN
 F 2 "modFiles:Resistor_small" V 3680 4800 50  0001 C CNN
 F 3 "~" H 3750 4800 50  0001 C CNN
@@
 P 3750 5150
 F 0 "R49" V 3830 5150 50  0000 C CNN
-F 1 "1K" V 3750 5150 50  0000 C CNN
+F 1 "100" V 3750 5150 50  0000 C CNN
 F 2 "modFiles:Resistor_small" V 3680 5150 50  0001 C CNN
 F 3 "~" H 3750 5150 50  0001 C CNN
@@
 P 3750 5500
 F 0 "R50" V 3830 5500 50  0000 C CNN
-F 1 "470" V 3750 5500 50  0000 C CNN
+F 1 "47" V 3750 5500 50  0000 C CNN
 F 2 "modFiles:Resistor_small" V 3680 5500 50  0001 C CNN
 F 3 "~" H 3750 5500 50  0001 C CNN
@@
 P 3750 5850
 F 0 "R51" V 3830 5850 50  0000 C CNN
-F 1 "330" V 3750 5850 50  0000 C CNN
+F 1 "33" V 3750 5850 50  0000 C CNN
 F 2 "modFiles:Resistor_small" V 3680 5850 50  0001 C CNN
 F 3 "~" H 3750 5850 50  0001 C CNN
@@
 P 3450 6000
 F 0 "R44" V 3530 6000 50  0000 C CNN
-F 1 "10K" V 3450 6000 50  0000 C CNN
+F 1 "1K" V 3450 6000 50  0000 C CNN
 F 2 "modFiles:Resistor_small" V 3380 6000 50  0001 C CNN
 F 3 "~" H 3450 6000 50  0001 C CNN
@@
 F 0 "Q6" H 14441 2896 50  0001 L CNN
 F 1 "BC547" H 13950 3050 50  0000 L CNN
-F 2 "Package_TO_SOT_THT:TO-92_Inline" H 14450 2775 50  0001 L CIN
+F 2 "modFiles:BC547" H 14450 2775 50  0001 L CIN
 F 3 "http://www.fairchildsemi.com/ds/BC/BC547.pdf" H 14250 2850 50  0001 L CNN
 	1    14250 2850
@@
 F 0 "Q5" H 13441 2896 50  0001 L CNN
 F 1 "BC547" H 12950 3050 50  0000 L CNN
-F 2 "Package_TO_SOT_THT:TO-92_Inline" H 13450 2775 50  0001 L CIN
+F 2 "modFiles:BC547" H 13450 2775 50  0001 L CIN
 F 3 "http://www.fairchildsemi.com/ds/BC/BC547.pdf" H 13250 2850 50  0001 L CNN
 	1    13250 2850
@@
 F 0 "Q7" H 14541 1846 50  0001 L CNN
 F 1 "BC547" H 14050 2000 50  0000 L CNN
-F 2 "Package_TO_SOT_THT:TO-92_Inline" H 14550 1725 50  0001 L CIN
+F 2 "modFiles:BC547" H 14550 1725 50  0001 L CIN
 F 3 "http://www.fairchildsemi.com/ds/BC/BC547.pdf" H 14350 1800 50  0001 L CNN
 	1    14350 1800
@@
 	1    0    0    -1
 $EndComp
+Wire Wire Line
+	6550 6100 6600 6100
+Connection ~ 6550 6100
+Text Label 6600 6100 0    50   ~ 0
+Z
+Wire Wire Line
+	13850 1600 13900 1600
+Connection ~ 13850 1600
+Text Label 13900 1600 0    50   ~ 0
+B_Z
+$Comp
+L Device:R R66
+U 1 1 5F53FF9B
+P 4400 1400
+F 0 "R66" H 4470 1446 50  0000 L CNN
+F 1 "R" H 4470 1355 50  0000 L CNN
+F 2 "modFiles:Resistor_small" V 4330 1400 50  0001 C CNN
+F 3 "~" H 4400 1400 50  0001 C CNN
+	1    4400 1400
+	0    1    1    0
+$EndComp
+Wire Wire Line
+	4250 1200 4250 1400
+Wire Wire Line
+	4550 1400 4550 1250
+Wire Wire Line
+	4550 1250 4700 1250
+Wire Wire Line
+	4700 1250 4700 1100
+Connection ~ 4700 1100
+Wire Wire Line
+	4700 1100 4600 1100
+$Comp
+L Device:R R74
+U 1 1 5F5CB460
+P 4550 900
+F 0 "R74" H 4620 946 50  0000 L CNN
+F 1 "R" H 4620 855 50  0000 L CNN
+F 2 "modFiles:Resistor_small" V 4480 900 50  0001 C CNN
+F 3 "~" H 4550 900 50  0001 C CNN
+	1    4550 900
+	0    1    1    0
+$EndComp
+Wire Wire Line
+	4700 900  4850 900
+Wire Wire Line
+	4400 900  4250 900
+Connection ~ 4250 900
 $EndSCHEMATC

Commit message: finalized board
Parts:
- added J13: Conn_01x01_Female, Connector_PinHeader_2.00mm:PinHeader_1x01_P2.00mm_Vertical, symbol Connector:Conn_01x01_Female
Connections:
- net Z: now also J13.1 (Pin_1)
Changed lines of the file:
@@
 	4400 900  4250 900
 Connection ~ 4250 900
+$Comp
+L Connector:Conn_01x01_Female J13
+U 1 1 5F42F269
+P 10450 4550
+F 0 "J13" H 10477 4576 50  0000 L CNN
+F 1 "Conn_01x01_Female" H 10477 4485 50  0000 L CNN
+F 2 "Connector_PinHeader_2.00mm:PinHeader_1x01_P2.00mm_Vertical" H 10450 4550 50  0001 C CNN
+F 3 "~" H 10450 4550 50  0001 C CNN
+	1    10450 4550
+	1    0    0    -1
+$EndComp
+Text Label 10250 4550 2    50   ~ 0
+Z
 $EndSCHEMATC
